Commit message: Update arm_moveit_config and image_pose_tracking configurations and files for improved functionality and structure

File: image_pose_tracking/config/right_arm_baseline.urdf (robot description, URDF)
Before this commit: robot upper_arm, 10 links, 9 joints
Joints:
- joint jRightWrist_rotz: limit lower=-0.523599 upper=0.349066 effort=30 velocity=1.0 -> lower=-1.57 upper=1.57 effort=30 velocity=1.0

File: image_pose_tracking/config/right_arm_red.urdf (robot description, URDF)
Before this commit: robot upper_arm, 9 links, 8 joints
Links:
- added link RightHandCOM, mass 0.00001; visual box size=0 0 0
Joints:
- added joint jRightHandCOM: type fixed, parent RightHand, child RightHandCOM, origin xyz=0 -0.096206 0 rpy=0 0 0, axis 0 0 0
- joint world_to_shoulder: origin xyz=-0.0361881  -0.14083758  1.01600003 rpy=3.14 1.57 0 -> xyz=-0.02348199 -0.12654904  1.02600002 rpy=3.14 1.57 0
