Commit message: Enhance MediaPipe Pose Node with Joint State Subscription and Danger Zone Indicators
- Added subscription to JointState messages for optimized arm joint states.
- Implemented danger zone checks for elbow, shoulder, and wrist based on joint angles.
- Updated image publishing to include visual indicators for danger zones on the annotated image.
- Adjusted point cloud extraction to offset the x-coordinate of the first valid point.
- Updated package.xml to include new dependencies.
- Modified setup.py to include additional URDF files in the package.
- Changed static transformation parameters in joint velocity estimation configuration.
- Refactored joint velocity estimator to streamline camera to shoulder transformation initialization.
- Updated pose optimization parameters for improved optimization performance.
- Replaced URDF model in pose optimizer with a new optimized version.
- Removed realsense-ros submodule.
- Added ground truth and optimized URDF configurations for the right arm.

File: image_pose_tracking/config/right_arm_gt.urdf (robot description, URDF)
Before this commit: robot upper_arm, 11 links, 10 joints
Links:
- removed link RightForeArm
- removed link RightForeArm_f1
- removed link RightHand
- removed link RightHandCOM
- removed link RightHand_f1
- removed link RightShoulder
- removed link RightUpperArm
- removed link RightUpperArm_f1
- removed link RightUpperArm_f2
- removed link Trunk
- added link gt_RightForeArm, mass 1.454; collision cylinder length=0.248 radius=0.02; visual cylinder length=0.248 radius=0.02
- added link gt_RightForeArm_f1, mass 0; visual sphere radius=0.02
- added link gt_RightHand, mass 0.4362; collision box size=0.04 0.133 0.133; visual box size=0.06 0.085 0.03
- added link gt_RightHandCOM, mass 0.00001; visual box size=0 0 0
- added link gt_RightHand_f1, mass 0
- added link gt_RightShoulder; visual sphere radius=0.02
- added link gt_RightUpperArm, mass 2.181; collision cylinder length=0.299 radius=0.02; visual cylinder length=0.299 radius=0.02
- added link gt_RightUpperArm_f1, mass 0
- added link gt_RightUpperArm_f2, mass 0
- added link gt_Trunk, mass 5.0; collision cylinder length=0.4 radius=0.02; visual cylinder length=0.4 radius=0.02
Joints:
- removed joint jRightElbow_roty
- removed joint jRightElbow_rotz
- removed joint jRightHandCOM
- removed joint jRightShoulder_rotx
- removed joint jRightShoulder_roty
- removed joint jRightShoulder_rotz
- removed joint jRightWrist_rotx
- removed joint jRightWrist_rotz
- removed joint jShoulder_to_trunk
- removed joint world_to_shoulder
- added joint gt_jRightElbow_roty: type revolute, parent gt_RightForeArm, child gt_RightForeArm_f1, origin xyz=0 -0.248 0 rpy=0 0 0, axis 0 1 0, limit lower=-1.5708 upper=1.48353 effort=30 velocity=1.0
- added joint gt_jRightElbow_rotz: type revolute, parent gt_RightUpperArm, child gt_RightForeArm, origin xyz=0 -0.299 0 rpy=0 0 0, axis 0 0 1, limit lower=0 upper=2.53073 effort=30 velocity=1.0
- added joint gt_jRightHand_COM: type fixed, parent gt_RightHand, child gt_RightHandCOM, origin xyz=0 -0.07 0 rpy=0 0 0, axis 0 0 0
- added joint gt_jRightShoulder_rotx: type revolute, parent gt_RightShoulder, child gt_RightUpperArm_f1, origin xyz=0 0 0 rpy=0 0 0, axis 1 0 0, limit lower=-2.35619 upper=1.5708 effort=30 velocity=1.0
- added joint gt_jRightShoulder_roty: type revolute, parent gt_RightUpperArm_f2, child gt_RightUpperArm, origin xyz=0 0 0 rpy=0 0 0, axis 0 1 0, limit lower=-1.5708 upper=1.5708 effort=30 velocity=1.0
- added joint gt_jRightShoulder_rotz: type revolute, parent gt_RightUpperArm_f1, child gt_RightUpperArm_f2, origin xyz=0 0 0 rpy=0 0 0, axis 0 0 1, limit lower=-0.785398 upper=1.5708 effort=30 velocity=1.0
- added joint gt_jRightWrist_rotx: type revolute, parent gt_RightForeArm_f1, child gt_RightHand_f1, origin xyz=0    0  0 rpy=0 0 0, axis 1 0 0, limit lower=-1.5708 upper=1.5708 effort=30 velocity=1.0
- added joint gt_jRightWrist_rotz: type revolute, parent gt_RightHand_f1, child gt_RightHand, origin xyz=0 0 0 rpy=0 0 0, axis 0 0 1, limit lower=-0.723599 upper=0.549066 effort=30 velocity=1.0
- added joint gt_jShoulder_to_trunk: type fixed, parent gt_RightShoulder, child gt_Trunk, origin xyz=0 0 -0.20 rpy=0 0 0
- added joint gt_world_to_shoulder: type fixed, parent camera_depth_optical_frame, child gt_RightShoulder, origin xyz=-0.12466341 -0.152376    1.07400005 rpy=3.14 1.57 0

File: image_pose_tracking/config/right_arm_opt.urdf (robot description, URDF)
Before this commit: robot upper_arm, 11 links, 10 joints
Links:
- removed link RightForeArm
- removed link RightForeArm_f1
- removed link RightHand
- removed link RightHandCOM
- removed link RightHand_f1
- removed link RightShoulder
- removed link RightUpperArm
- removed link RightUpperArm_f1
- removed link RightUpperArm_f2
- removed link Trunk
- added link opt_RightForeArm, mass 1.454; collision cylinder length=0.248 radius=0.02; visual cylinder length=0.248 radius=0.02
- added link opt_RightForeArm_f1, mass 0; visual sphere radius=0.02
- added link opt_RightHand, mass 0.4362; collision box size=0.04 0.133 0.133; visual box size=0.06 0.085 0.03
- added link opt_RightHandCOM, mass 0.00001; visual box size=0 0 0
- added link opt_RightHand_f1, mass 0
- added link opt_RightShoulder; visual sphere radius=0.02
- added link opt_RightUpperArm, mass 2.181; collision cylinder length=0.299 radius=0.02; visual cylinder length=0.299 radius=0.02
- added link opt_RightUpperArm_f1, mass 0
- added link opt_RightUpperArm_f2, mass 0
- added link opt_Trunk, mass 5.0; collision cylinder length=0.4 radius=0.02; visual cylinder length=0.4 radius=0.02
Joints:
- removed joint jRightElbow_roty
- removed joint jRightElbow_rotz
- removed joint jRightHandCOM
- removed joint jRightShoulder_rotx
- removed joint jRightShoulder_roty
- removed joint jRightShoulder_rotz
- removed joint jRightWrist_rotx
- removed joint jRightWrist_rotz
- removed joint jShoulder_to_trunk
- removed joint world_to_shoulder
- added joint opt_jRightElbow_roty: type revolute, parent opt_RightForeArm, child opt_RightForeArm_f1, origin xyz=0 -0.248 0 rpy=0 0 0, axis 0 1 0, limit lower=-1.5708 upper=1.48353 effort=30 velocity=1.0
- added joint opt_jRightElbow_rotz: type revolute, parent opt_RightUpperArm, child opt_RightForeArm, origin xyz=0 -0.299 0 rpy=0 0 0, axis 0 0 1, limit lower=0 upper=2.53073 effort=30 velocity=1.0
- added joint opt_jRightHand_COM: type fixed, parent opt_RightHand, child opt_RightHandCOM, origin xyz=0 -0.07 0 rpy=0 0 0, axis 0 0 0
- added joint opt_jRightShoulder_rotx: type revolute, parent opt_RightShoulder, child opt_RightUpperArm_f1, origin xyz=0 0 0 rpy=0 0 0, axis 1 0 0, limit lower=-2.35619 upper=1.5708 effort=30 velocity=1.0
- added joint opt_jRightShoulder_roty: type revolute, parent opt_RightUpperArm_f2, child opt_RightUpperArm, origin xyz=0 0 0 rpy=0 0 0, axis 0 1 0, limit lower=-1.5708 upper=1.5708 effort=30 velocity=1.0
- added joint opt_jRightShoulder_rotz: type revolute, parent opt_RightUpperArm_f1, child opt_RightUpperArm_f2, origin xyz=0 0 0 rpy=0 0 0, axis 0 0 1, limit lower=-0.785398 upper=1.5708 effort=30 velocity=1.0
- added joint opt_jRightWrist_rotx: type revolute, parent opt_RightForeArm_f1, child opt_RightHand_f1, origin xyz=0    0  0 rpy=0 0 0, axis 1 0 0, limit lower=-1.5708 upper=1.5708 effort=30 velocity=1.0
- added joint opt_jRightWrist_rotz: type revolute, parent opt_RightHand_f1, child opt_RightHand, origin xyz=0 0 0 rpy=0 0 0, axis 0 0 1, limit lower=-0.723599 upper=0.549066 effort=30 velocity=1.0
- added joint opt_jShoulder_to_trunk: type fixed, parent opt_RightShoulder, child opt_Trunk, origin xyz=0 0 -0.20 rpy=0 0 0
- added joint opt_world_to_shoulder: type fixed, parent camera_depth_optical_frame, child opt_RightShoulder, origin xyz=-0.12466341 -0.152376    1.07400005 rpy=3.14 1.57 0
