Commit message: Add std_msgs dependency and update joint state handling
- Added std_msgs as a required package in CMakeLists.txt and package.xml.
- Updated parameters.yaml with new translation and rotation values for ee2hand.
- Changed joint_state_callback to use Float32MultiArray instead of JointState.
- Adjusted cost function to accommodate changes in joint state representation.
- Implemented velocity smoothing logic in the optimizer.
- Introduced a new URDF file for the right arm configuration.

File: image_pose_tracking/config/right_arm_upt.urdf (robot description, URDF)
Before this commit: robot upper_arm, 13 links, 12 joints
Links:
- removed link Head
- removed link Neck
- removed link T8
- removed link gt_RightForeArm
- removed link gt_RightForeArm_f1
- removed link gt_RightHand
- removed link gt_RightHandCOM
- removed link gt_RightHand_f1
- removed link gt_RightShoulder
- removed link gt_RightUpperArm
- removed link gt_RightUpperArm_f1
- removed link gt_RightUpperArm_f2
- added link upt_RightForeArm, mass 1.454; collision cylinder length=0.248 radius=0.02; visual cylinder length=0.248 radius=0.02
- added link upt_RightForeArm_f1, mass 0; visual sphere radius=0.02
- added link upt_RightHand, mass 0.4362; collision box size=0.04 0.133 0.133; visual box size=0.06 0.085 0.03
- added link upt_RightHandCOM, mass 0.00001; visual box size=0 0 0
- added link upt_RightHand_f1, mass 0
- added link upt_RightShoulder; visual sphere radius=0.02
- added link upt_RightUpperArm, mass 2.181; collision cylinder length=0.299 radius=0.02; visual cylinder length=0.299 radius=0.02
- added link upt_RightUpperArm_f1, mass 0
- added link upt_RightUpperArm_f2, mass 0
- added link upt_Trunk, mass 5.0; collision cylinder length=0.4 radius=0.02; visual cylinder length=0.4 radius=0.02
Joints:
- removed joint gt_jRightElbow_roty
- removed joint gt_jRightElbow_rotz
- removed joint gt_jRightHand_COM
- removed joint gt_jRightShoulder_rotx
- removed joint gt_jRightShoulder_roty
- removed joint gt_jRightShoulder_rotz
- removed joint gt_jRightWrist_rotx
- removed joint gt_jRightWrist_rotz
- removed joint gt_world_to_shoulder
- removed joint jHead
- removed joint jNeck
- removed joint jTrunk
- added joint upt_jRightElbow_roty: type revolute, parent upt_RightForeArm, child upt_RightForeArm_f1, origin xyz=0 -0.248 0 rpy=0 0 0, axis 0 1 0, limit lower=-1.5708 upper=1.48353 effort=30 velocity=1.0
- added joint upt_jRightElbow_rotz: type revolute, parent upt_RightUpperArm, child upt_RightForeArm, origin xyz=0 -0.299 0 rpy=0 0 0, axis 0 0 1, limit lower=0 upper=2.53073 effort=30 velocity=1.0
- added joint upt_jRightHand_COM: type fixed, parent upt_RightHand, child upt_RightHandCOM, origin xyz=0 -0.07 0 rpy=0 0 0, axis 0 0 0
- added joint upt_jRightShoulder_rotx: type revolute, parent upt_RightShoulder, child upt_RightUpperArm_f1, origin xyz=0 0 0 rpy=0 0 0, axis 1 0 0, limit lower=-2.35619 upper=1.5708 effort=30 velocity=1.0
- added joint upt_jRightShoulder_roty: type revolute, parent upt_RightUpperArm_f2, child upt_RightUpperArm, origin xyz=0 0 0 rpy=0 0 0, axis 0 1 0, limit lower=-1.5708 upper=1.5708 effort=30 velocity=1.0
- added joint upt_jRightShoulder_rotz: type revolute, parent upt_RightUpperArm_f1, child upt_RightUpperArm_f2, origin xyz=0 0 0 rpy=0 0 0, axis 0 0 1, limit lower=-0.785398 upper=1.5708 effort=30 velocity=1.0
- added joint upt_jRightWrist_rotx: type revolute, parent upt_RightForeArm_f1, child upt_RightHand_f1, origin xyz=0    0  0 rpy=0 0 0, axis 1 0 0, limit lower=-1.5708 upper=1.5708 effort=30 velocity=1.0
- added joint upt_jRightWrist_rotz: type revolute, parent upt_RightHand_f1, child upt_RightHand, origin xyz=0 0 0 rpy=0 0 0, axis 0 0 1, limit lower=-0.723599 upper=0.549066 effort=30 velocity=1.0
- added joint upt_jShoulder_to_trunk: type fixed, parent upt_RightShoulder, child upt_Trunk, origin xyz=0 0 -0.20 rpy=0 0 0
- added joint upt_world_to_shoulder: type fixed, parent camera_depth_optical_frame, child upt_RightShoulder, origin xyz=-0.12466341 -0.152376    1.07400005 rpy=3.14 1.57 0
