Commit message: Refactor arm_moveit_config and ik_solver_moveit packages
- Updated URDF files for right arm configuration with new joint origins and added RightHandCOM link.
- Created new MoveIt configuration package for upper arm with necessary launch files and configuration settings.
- Implemented kinematics and joint limits configuration for the arm.
- Developed inverse kinematics solver in ik_solver_moveit package to compute joint states based on end-effector pose.
- Added parameter configuration for end-effector to hand transformation and operational settings for optimization.
- Enhanced launch files for better integration with MoveIt and ROS 2 ecosystem.

File: image_pose_tracking/config/right_arm.urdf (robot description, URDF)
Before this commit: robot upper_arm, 9 links, 8 joints
Joints:
- joint world_to_shoulder: origin xyz=-0.05723638 -0.11301016  1.0710001 rpy=3.14 1.57 0 -> xyz=-0.0361881  -0.14083758  1.01600003 rpy=3.14 1.57 0

File: image_pose_tracking/config/right_arm_red.urdf (robot description, URDF)
Before this commit: robot upper_arm, 9 links, 8 joints
Joints:
- joint world_to_shoulder: origin xyz=-0.05723638 -0.11301016  1.0710001 rpy=3.14 1.57 0 -> xyz=-0.0361881  -0.14083758  1.01600003 rpy=3.14 1.57 0

Commit message: feat: Integrate NLopt optimization method into pose optimization
- Updated CMakeLists.txt to include NLopt as a dependency and added main.cpp for executable entry point.
- Modified parameters.yaml to switch optimization method to NLopt and added relevant parameters for NLopt configuration.
- Refactored optimizer.cpp to implement NLopt optimization alongside existing SVD method, including cost function and joint state handling.
- Introduced new header file optimizer.hpp to define PoseOptimizer class and encapsulate related functionalities.
- Enhanced error handling and logging for optimization processes.

File: image_pose_tracking/config/right_arm.urdf (robot description, URDF)
Before this commit: robot upper_arm, 10 links, 9 joints
Joints:
- joint jRightHandCOM: origin xyz=0 -0.096206 0 rpy=0 0 0 -> xyz=0 -0.05 0 rpy=0 0 0
- joint world_to_shoulder: origin xyz=-0.02348199 -0.12654904  1.02600002 rpy=3.14 1.57 0 -> xyz=-0.03230042 -0.11765296  1.16500001 rpy=3.14 1.57 0

File: image_pose_tracking/config/right_arm_baseline.urdf (robot description, URDF)
Before this commit: robot upper_arm, 10 links, 9 joints
Joints:
- joint jRightHandCOM: origin xyz=0 -0.096206 0 rpy=0 0 0 -> xyz=0 -0.05 0 rpy=0 0 0
- joint world_to_shoulder: origin xyz=-0.02348199 -0.12654904  1.02600002 rpy=3.14 1.57 0 -> xyz=-0.03230042 -0.11765296  1.16500001 rpy=3.14 1.57 0

File: image_pose_tracking/config/right_arm_red.urdf (robot description, URDF)
Before this commit: robot upper_arm, 10 links, 9 joints
Joints:
- joint jRightHandCOM: origin xyz=0 -0.096206 0 rpy=0 0 0 -> xyz=0 -0.05 0 rpy=0 0 0
- joint world_to_shoulder: origin xyz=-0.02348199 -0.12654904  1.02600002 rpy=3.14 1.57 0 -> xyz=-0.03230042 -0.11765296  1.16500001 rpy=3.14 1.57 0

Commit message: commit before kalman filter velocity

File: image_pose_tracking/config/right_arm.urdf (robot description, URDF)
Before this commit: robot upper_arm, 10 links, 9 joints
Links:
- link RightForeArm: geometry collision cylinder length=0.224 radius=0.023721; visual cylinder length=0.224 radius=0.023721
- link RightUpperArm: geometry collision cylinder length=0.25 radius=0.035581; visual cylinder length=0.25 radius=0.035581
Joints:
- joint jRightElbow_roty: origin xyz=0 -0.27 0 rpy=0 0 0 -> xyz=0 -0.224 0 rpy=0 0 0
- joint jRightElbow_rotz: origin xyz=0 -0.24 0 rpy=0 0 0 -> xyz=0 -0.25 0 rpy=0 0 0

Commit message: feat: Update arm solver parameters and enhance sensitivity analysis configuration

File: image_pose_tracking/config/right_arm.urdf (robot description, URDF)
Before this commit: robot upper_arm, 11 links, 10 joints
Joints:
- joint world_to_shoulder: origin xyz=-0.12466341 -0.152376    1.07400005 rpy=3.14 1.57 0 -> xyz=-0.10466341 -0.122376    1.07400005 rpy=3.14 1.57 0

File: image_pose_tracking/config/right_arm_gt.urdf (robot description, URDF)
Before this commit: robot upper_arm, 13 links, 12 joints
Joints:
- joint gt_world_to_shoulder: origin xyz=-0.12466341 -0.152376    1.07400005 rpy=3.14 1.57 0 -> xyz=-0.10466341 -0.122376    1.07400005 rpy=3.14 1.57 0

File: image_pose_tracking/config/right_arm_opt.urdf (robot description, URDF)
Before this commit: robot upper_arm, 11 links, 10 joints
Joints:
- joint opt_world_to_shoulder: origin xyz=-0.12466341 -0.152376    1.07400005 rpy=3.14 1.57 0 -> xyz=-0.10466341 -0.122376    1.07400005 rpy=3.14 1.57 0

File: image_pose_tracking/config/right_arm_upt.urdf (robot description, URDF)
Before this commit: robot upper_arm, 11 links, 10 joints
Joints:
- joint upt_world_to_shoulder: origin xyz=-0.12466341 -0.152376    1.07400005 rpy=3.14 1.57 0 -> xyz=-0.10466341 -0.122376    1.07400005 rpy=3.14 1.57 0

Commit message: feat: Implement sensitivity analysis in joint velocity estimation and pose optimization

File: image_pose_tracking/config/right_arm.urdf (robot description, URDF)
Before this commit: robot upper_arm, 11 links, 10 joints
Joints:
- joint world_to_shoulder: origin xyz=-0.10466341 -0.122376    1.07400005 rpy=3.14 1.57 0 -> xyz=-0.10466341 -0.122376    1.00400005 rpy=3.14 1.57 0

File: image_pose_tracking/config/right_arm_gt.urdf (robot description, URDF)
Before this commit: robot upper_arm, 13 links, 12 joints
Joints:
- joint gt_world_to_shoulder: origin xyz=-0.10466341 -0.122376    1.07400005 rpy=3.14 1.57 0 -> xyz=-0.10466341 -0.122376    1.00400005 rpy=3.14 1.57 0

File: image_pose_tracking/config/right_arm_opt.urdf (robot description, URDF)
Before this commit: robot upper_arm, 11 links, 10 joints
Joints:
- joint opt_world_to_shoulder: origin xyz=-0.10466341 -0.122376    1.07400005 rpy=3.14 1.57 0 -> xyz=-0.10466341 -0.122376    1.00400005 rpy=3.14 1.57 0

File: image_pose_tracking/config/right_arm_upt.urdf (robot description, URDF)
Before this commit: robot upper_arm, 11 links, 10 joints
Joints:
- joint upt_world_to_shoulder: origin xyz=-0.10466341 -0.122376    1.07400005 rpy=3.14 1.57 0 -> xyz=-0.10466341 -0.122376    1.00400005 rpy=3.14 1.57 0

Commit message: fix: Mark subprojects as dirty to indicate uncommitted changes

File: image_pose_tracking/config/right_arm.urdf (robot description, URDF)
Before this commit: robot upper_arm, 11 links, 10 joints
Links:
- removed link camera_depth_optical_frame
Joints:
- removed joint world_to_shoulder

File: image_pose_tracking/config/right_arm.urdf.xacro (robot description, xacro)
@@ -1,28 +1,36 @@
-<robot name="upper_arm">
+<?xml version="1.0"?>
+<robot xmlns:xacro="http://www.ros.org/wiki/xacro" name="upper_arm">
+    <xacro:property name="prefix" value="$(arg robot_prefix)"/>
+    <xacro:property name="color" value="$(arg robot_color)"/>
+    <xacro:property name="color_code"  value="${
+        '0.35 0.55 0.40 1' if color == 'green'
+        else '0.25 0.45 0.65 1' if color == 'blue'
+        else '0.72 0.70 0.65 1'}"/>
     <material name="color">
-        <color rgba="0 1 0 1"/>
+        <color rgba="${color_code}"/>
     </material>
-    <link name="camera_depth_optical_frame"/>
-    <joint name="gt_world_to_shoulder" type="fixed">
+    <!-- <link name="camera_depth_optical_frame"/> -->
+    <!-- <joint name="${prefix}world_to_shoulder" type="fixed">
         <parent link="camera_depth_optical_frame"/>
-        <child link="gt_RightShoulder"/>
+        <child link="${prefix}RightShoulder"/>
         <origin xyz="-0.10466341 -0.122376    1.00400005" rpy="3.14 1.57 0"/>
-        <!-- y motion -->
-        <!-- <origin xyz="-0.10466341 -0.122376    1.02" rpy="3.14 1.57 0"/> -->
-        <!-- z motion -->
-    </joint>
+    </joint> -->
         <!-- === Trunk slab (torso) === -->
-    <link name="T8">
-        <inertial>
+    <link name="${prefix}Trunk">
+        <inertial>
+            <!-- Give it a small but nonzero mass to avoid NaNs -->
             <mass value="5.0"/>
             <origin xyz="0 0 0.20" rpy="0 0 0"/>
+            <!-- Rough, diagonal-dominant inertia for a 0.40 x 0.25 x 0.55 m box -->
             <inertia ixx="0.5" iyy="0.8" izz="0.5" ixy="0" ixz="0" iyz="0"/>
         </inertial>
         <visual>
             <origin xyz="0 0 0" rpy="0 0 0"/>
-            <geometry>
-                <cylinder length="0.4" radius="0.05"/>
+            <!-- size = [width_x, depth_y, height_z] -->
+            <geometry>
+                <cylinder length="0.4" radius="0.02"/>
             </geometry>
             <material name="color">
+                <!-- subtle gray so the arm (green) stands out -->
                 <color rgba="0.6 0.6 0.6 1.0"/>
             </material>
@@ -31,141 +39,58 @@
             <origin xyz="0 0 0" rpy="0 0 0"/>
             <geometry>
-                <cylinder length="0.4" radius="0.05"/>
-            </geometry>
-        </collision>
-    </link>
-    <link name="Neck">
-        <inertial>
-            <mass value="0.8724"/>
-			<!--COM origin wrt jT1C7-->
-            <origin xyz="0  0 0" rpy="1.57 0 0" />
-            <inertia ixx="0.00091024" iyy="0.00091024" izz="0.00043345" ixy="0" ixz="0" iyz="0"/>
-        </inertial>
-        <visual>
-			<!--box origin wrt jT1C7-->
-            <origin xyz="0    0.0 0" rpy="1.57 0 0" />
-            <geometry>
-		<cylinder length="0.1" radius="0.05"/>
-            </geometry>
-            <material name="color"/>
-        </visual>
-        <collision>
-			<!--box origin wrt jT1C7-->
-            <origin xyz="0    0.0 0" rpy="1.57 0 0" />
-            <geometry>
-                <cylinder length="0.1" radius="0.05"/>
-            </geometry>
-        </collision>
-    </link>
-    <link name="Head">
-        <inertial>
-            <mass value="2.6172"/>
-			<!--COM origin wrt jC1Head-->
-            <origin xyz="0           0    0" rpy="0 0 0" />
-            <inertia ixx="0.010376" iyy="0.010376" izz="0.010376" ixy="0" ixz="0" iyz="0"/>
-        </inertial>
-        <visual>
-			<!--boc origin wrt jC1Head-->
-            <origin xyz="0           0    0" rpy="0 0 0" />
-            <geometry>
-                <sphere radius="0.1"/>
-            </geometry>
-            <material name="color"/>
-        </visual>
-        <collision>
-			<!--box origin wrt jC1Head-->
-            <origin xyz="0           0    0" rpy="0 0 0" />
-            <geometry>
-                <sphere radius="0.1"/>
-            </geometry>
-        </collision>
-    </link>
-    <joint name="jTrunk" type="fixed">
-        <origin xyz="0 0 -0.2" rpy="0 0 0"/>
-        <parent link="gt_RightShoulder"/>
-        <child link="T8"/>
-    </joint>
-    <joint name="jNeck" type="fixed">
-        <origin xyz="0  0.05 0" rpy="0 0 0"/>
-        <parent link="T8"/>
-        <child link="Neck"/>
-    </joint>
-    <joint name="jHead" type="fixed">
-        <origin xyz="0 0.1 0" rpy="0 0 0"/>
-        <parent link="Neck"/>
-        <child link="Head"/>
-    </joint>
-    <!-- <link name="gt_Trunk">
-        <inertial>
-            <mass value="5.0"/>
-            <origin xyz="0 0 0.20" rpy="0 0 0"/>
-            <inertia ixx="0.5" iyy="0.8" izz="0.5" ixy="0" ixz="0" iyz="0"/>
-        </inertial>
-        <visual>
-            <origin xyz="0 0 0" rpy="0 0 0"/>
-            <geometry>
                 <cylinder length="0.4" radius="0.02"/>
             </geometry>
-            <material name="color">
-                <color rgba="0.6 0.6 0.6 1.0"/>
-            </material>
-        </visual>
-        <collision>
-            <origin xyz="0 0 0" rpy="0 0 0"/>
-            <geometry>
-                <cylinder length="0.4" radius="0.02"/>
-            </geometry>
-        </collision>
-    </link> -->
-    <!-- <joint name="gt_jShoulder_to_trunk" type="fixed">
+        </collision>
+    </link>
+    <joint name="${prefix}jShoulder_to_trunk" type="fixed">
         <origin xyz="0 0 -0.20" rpy="0 0 0"/>
-        <parent link="gt_RightShoulder"/>
-        <child link="gt_Trunk"/>
-    </joint> -->
+        <parent link="${prefix}RightShoulder"/>
+        <child link="${prefix}Trunk"/>
+    </joint>
     <!--  shoudler, 3DOF -->
-    <link name="gt_RightShoulder">
+    <link name="${prefix}RightShoulder">
         <visual>
 			<!--box origin wrt jRightC7Shoulder. RPY rotated of pi/2.-->
             <origin xyz="0 0 0" rpy="0 0 0" />
             <geometry>
-                <sphere radius="0.05"/>
-            </geometry>
-            <material name="color"/>
-        </visual>
-    </link>
-    <joint name="gt_jRightShoulder_rotx" type="revolute">
-        <origin xyz="0 0 0" rpy="0 0 0"/>
-        <parent link="gt_RightShoulder"/>
-        <child link="gt_RightUpperArm_f1"/>
+                <sphere radius="0.02"/>
+            </geometry>
+            <material name="color"/>
+        </visual>
+    </link>
+    <joint name="${prefix}jRightShoulder_rotx" type="revolute">
+        <origin xyz="0 0 0" rpy="0 0 0"/>
+        <parent link="${prefix}RightShoulder"/>
+        <child link="${prefix}RightUpperArm_f1"/>
         <dynamics damping="0.1" friction="0.0"/>
         <limit effort="30" velocity="1.0" lower="-2.35619" upper="1.5708" />
         <axis xyz="1 0 0" />
     </joint>
-    <link name="gt_RightUpperArm_f1">
-        <inertial>
-            <mass value="0"/>
-            <origin xyz="0 0 0" rpy="0 0 0" />
-            <inertia ixx="0" iyy="0" izz="0" ixy="0" ixz="0" iyz="0"/>
-        </inertial>
-    </link>
-    <joint name="gt_jRightShoulder_rotz" type="revolute">
-        <origin xyz="0 0 0" rpy="0 0 0"/>
-        <parent link="gt_RightUpperArm_f1"/>
-        <child link="gt_RightUpperArm_f2"/>
+    <link name="${prefix}RightUpperArm_f1">
+        <inertial>
+            <mass value="0"/>
+            <origin xyz="0 0 0" rpy="0 0 0" />
+            <inertia ixx="0" iyy="0" izz="0" ixy="0" ixz="0" iyz="0"/>
+        </inertial>
+    </link>
+    <joint name="${prefix}jRightShoulder_rotz" type="revolute">
+        <origin xyz="0 0 0" rpy="0 0 0"/>
+        <parent link="${prefix}RightUpperArm_f1"/>
+        <child link="${prefix}RightUpperArm_f2"/>
         <dynamics damping="0.1" friction="0.0"/>
         <limit effort="30" velocity="1.0" lower="-0.785398" upper="1.5708" />
         <axis xyz="0 0 1" />
     </joint>
-    <link name="gt_RightUpperArm_f2">
-        <inertial>
-            <mass value="0"/>
-            <origin xyz="0 0 0" rpy="0 0 0" />
-            <inertia ixx="0" iyy="0" izz="0" ixy="0" ixz="0" iyz="0"/>
-        </inertial>
-    </link>
-    <joint name="gt_jRightShoulder_roty" type="revolute">
-        <origin xyz="0 0 0" rpy="0 0 0"/>
-        <parent link="gt_RightUpperArm_f2"/>
-        <child link="gt_RightUpperArm"/>
+    <link name="${prefix}RightUpperArm_f2">
+        <inertial>
+            <mass value="0"/>
+            <origin xyz="0 0 0" rpy="0 0 0" />
+            <inertia ixx="0" iyy="0" izz="0" ixy="0" ixz="0" iyz="0"/>
+        </inertial>
+    </link>
+    <joint name="${prefix}jRightShoulder_roty" type="revolute">
+        <origin xyz="0 0 0" rpy="0 0 0"/>
+        <parent link="${prefix}RightUpperArm_f2"/>
+        <child link="${prefix}RightUpperArm"/>
         <dynamics damping="0.1" friction="0.0"/>
         <limit effort="30" velocity="1.0" lower="-1.5708" upper="1.5708" />
@@ -173,9 +98,9 @@
     </joint>
     <!-- elbow, 3 dof -->
-    <link name="gt_RightUpperArm">
+    <link name="${prefix}RightUpperArm">
         <inertial>
             <mass value="2.181"/>
 			<!--COM origin wrt jRightShoulder-->
-            <origin xyz="0    -0.15         0" rpy="0 0 0" />
+            <origin xyz="0    -0.15           0" rpy="0 0 0" />
             <inertia ixx="0.020332" iyy="0.0013806" izz="0.020332" ixy="0" ixz="0" iyz="0"/>
         </inertial>
@@ -196,13 +121,13 @@
         </collision>
     </link>
-    <joint name="gt_jRightElbow_rotz" type="revolute">
+    <joint name="${prefix}jRightElbow_rotz" type="revolute">
         <origin xyz="0 -0.299 0" rpy="0 0 0"/>
-        <parent link="gt_RightUpperArm"/>
-        <child link="gt_RightForeArm"/>
+        <parent link="${prefix}RightUpperArm"/>
+        <child link="${prefix}RightForeArm"/>
         <dynamics damping="0.1" friction="0.0"/>
         <limit effort="30" velocity="1.0" lower="0" upper="2.53073" />
         <axis xyz="0 0 1" />
     </joint>
-    <link name="gt_RightForeArm">
+    <link name="${prefix}RightForeArm">
         <inertial>
             <mass value="1.454"/>
@@ -227,13 +152,13 @@
         </collision>
     </link>
-    <joint name="gt_jRightElbow_roty" type="revolute">
+    <joint name="${prefix}jRightElbow_roty" type="revolute">
         <origin xyz="0 -0.248 0" rpy="0 0 0"/>
-        <parent link="gt_RightForeArm"/>
-        <child link="gt_RightForeArm_f1"/>
+        <parent link="${prefix}RightForeArm"/>
+        <child link="${prefix}RightForeArm_f1"/>
         <dynamics damping="0.1" friction="0.0"/>
         <limit effort="30" velocity="1.0" lower="-1.5708" upper="1.48353" />
         <axis xyz="0 1 0" />
     </joint>
-    <link name="gt_RightForeArm_f1">
+    <link name="${prefix}RightForeArm_f1">
         <inertial>
             <mass value="0"/>
@@ -250,28 +175,28 @@
     </link>
     <!-- wrist 2 dofs -->
-    <joint name="gt_jRightWrist_rotx" type="revolute">
+    <joint name="${prefix}jRightWrist_rotx" type="revolute">
         <origin xyz="0    0  0" rpy="0 0 0"/>
-        <parent link="gt_RightForeArm_f1"/>
-        <child link="gt_RightHand_f1"/>
+        <parent link="${prefix}RightForeArm_f1"/>
+        <child link="${prefix}RightHand_f1"/>
         <dynamics damping="0.1" friction="0.0"/>
         <limit effort="30" velocity="1.0" lower="-1.5708" upper="1.5708" />
         <axis xyz="1 0 0" />
     </joint>
-    <link name="gt_RightHand_f1">
-        <inertial>
-            <mass value="0"/>
-            <origin xyz="0 0 0" rpy="0 0 0" />
-            <inertia ixx="0" iyy="0" izz="0" ixy="0" ixz="0" iyz="0"/>
-        </inertial>
-    </link>
-    <joint name="gt_jRightWrist_rotz" type="revolute">
-        <origin xyz="0 0 0" rpy="0 0 0"/>
-        <parent link="gt_RightHand_f1"/>
-        <child link="gt_RightHand"/>
+    <link name="${prefix}RightHand_f1">
+        <inertial>
+            <mass value="0"/>
+            <origin xyz="0 0 0" rpy="0 0 0" />
+            <inertia ixx="0" iyy="0" izz="0" ixy="0" ixz="0" iyz="0"/>
+        </inertial>
+    </link>
+    <joint name="${prefix}jRightWrist_rotz" type="revolute">
+        <origin xyz="0 0 0" rpy="0 0 0"/>
+        <parent link="${prefix}RightHand_f1"/>
+        <child link="${prefix}RightHand"/>
         <dynamics damping="0.1" friction="0.0"/>
         <limit effort="30" velocity="1.0" lower="-0.723599" upper="0.549066" />
         <axis xyz="0 0 1" />
     </joint>
-    <link name="gt_RightHand">
+    <link name="${prefix}RightHand">
         <inertial>
             <mass value="0.4362"/>
@@ -296,11 +221,11 @@
         </collision>
     </link>
-    <joint name="gt_jRightHand_COM" type="fixed">
+    <joint name="${prefix}jRightHandCOM" type="fixed">
         <origin xyz="0 -0.07 0" rpy="0 0 0"/>
-        <parent link="gt_RightHand"/>
-        <child link="gt_RightHandCOM"/>
+        <parent link="${prefix}RightHand"/>
+        <child link="${prefix}RightHandCOM"/>
         <axis xyz="0 0 0" />
     </joint>
-    <link name="gt_RightHandCOM">
+    <link name="${prefix}RightHandCOM">
         <inertial>
             <mass value="0.00001"/>
