Commit message: Refactor MediaPipePoseNode: Remove joint state monitoring and danger zone indicators
- Eliminated the subscription to joint states and associated danger checks for elbow, shoulder, and wrist angles in MediaPipePoseNode.
- Updated the image processing logic to remove visual indicators for danger zones.
- Adjusted the logging to reflect the changes in functionality.

Enhance pose optimization parameters and velocity estimation

- Updated parameters.yaml to modify translation and rotation values for ee2hand.
- Introduced new parameters for velocity estimation, including Kalman filter usage and timing configurations.
- Adjusted process noise and measurement noise values for improved accuracy in velocity estimation.

Refactor joint velocity estimator for improved state management

- Modified the predict and correct methods in joint_velocity_estimator to include new parameters for velocity decay and acceleration cap.
- Enhanced the handling of joint measurements and task velocity corrections.
- Improved error handling and logging for non-finite states in Kalman filter.

Update optimizer to support dynamic arm model rendering

- Added functionality to render the arm model from XACRO files with dynamic parameters for arm lengths and colors.
- Updated the optimizer to use the new arm model rendering logic.
- Adjusted frame names to be dynamic based on robot prefix.

General code cleanup and organization

- Removed unused variables and improved code readability across multiple files.
- Ensured consistent naming conventions and parameter handling throughout the codebase.

File: image_pose_tracking/config/right_arm.urdf.xacro (robot description, xacro)
@@ -3,4 +3,8 @@
     <xacro:property name="prefix" value="$(arg robot_prefix)"/>
     <xacro:property name="color" value="$(arg robot_color)"/>
+    <xacro:property name="upper_arm_length" value="$(arg upper_arm_length)"/>
+    <xacro:property name="upper_arm_com_y" value="${-float(upper_arm_length) / 2.0}"/>
+    <xacro:property name="forearm_length" value="$(arg forearm_length)"/>
+    <xacro:property name="forearm_com_y" value="${-float(forearm_length) / 2.0}"/>
     <xacro:property name="color_code"  value="${
         '0.35 0.55 0.40 1' if color == 'green'
@@ -102,12 +106,12 @@
             <mass value="2.181"/>
 			<!--COM origin wrt jRightShoulder-->
-            <origin xyz="0    -0.15           0" rpy="0 0 0" />
+            <origin xyz="0 ${upper_arm_com_y} 0" rpy="0 0 0" />
             <inertia ixx="0.020332" iyy="0.0013806" izz="0.020332" ixy="0" ixz="0" iyz="0"/>
         </inertial>
         <visual>
 			<!--box origin wrt jRightShoulder. RPY rotated of pi/2.-->
-            <origin xyz="0    -0.15           0" rpy="1.5708 0 0" />
-            <geometry>
-                <cylinder length="0.299" radius="0.02"/>
+            <origin xyz="0 ${upper_arm_com_y} 0" rpy="1.5708 0 0" />
+            <geometry>
+                <cylinder length="${upper_arm_length}" radius="0.02"/>
             </geometry>
             <material name="color"/>
@@ -115,12 +119,12 @@
         <collision>
 			<!--box origin wrt jRightShoulder. RPY rotated of pi/2.-->
-            <origin xyz="0    -0.15           0" rpy="1.5708 0 0" />
-            <geometry>
-                <cylinder length="0.299" radius="0.02"/>
+            <origin xyz="0 ${upper_arm_com_y} 0" rpy="1.5708 0 0" />
+            <geometry>
+                <cylinder length="${upper_arm_length}" radius="0.02"/>
             </geometry>
         </collision>
     </link>
     <joint name="${prefix}jRightElbow_rotz" type="revolute">
-        <origin xyz="0 -0.299 0" rpy="0 0 0"/>
+        <origin xyz="0 ${-float(upper_arm_length)} 0" rpy="0 0 0"/>
         <parent link="${prefix}RightUpperArm"/>
         <child link="${prefix}RightForeArm"/>
@@ -133,12 +137,12 @@
             <mass value="1.454"/>
 			<!--COM origin wrt jRightElbow-->
-            <origin xyz="0    -0.124           0" rpy="0 0 0" />
+            <origin xyz="0 ${forearm_com_y} 0" rpy="0 0 0" />
             <inertia ixx="0.008948" iyy="0.00040906" izz="0.008948" ixy="0" ixz="0" iyz="0"/>
         </inertial>
         <visual>
 			<!--box origin wrt jRightElbow. RPY rotated of pi/2.-->
-            <origin xyz="0    -0.124           0" rpy="1.5708 0 0" />
-            <geometry>
-                <cylinder length="0.248" radius="0.02"/>
+            <origin xyz="0 ${forearm_com_y} 0" rpy="1.5708 0 0" />
+            <geometry>
+                <cylinder length="${forearm_length}" radius="0.02"/>
             </geometry>
             <material name="color"/>
@@ -146,12 +150,12 @@
         <collision>
 			<!--box origin wrt jRightElbow. RPY rotated of pi/2.-->
-            <origin xyz="0    -0.124           0" rpy="1.5708 0 0" />
-            <geometry>
-                <cylinder length="0.248" radius="0.02"/>
+            <origin xyz="0 ${forearm_com_y} 0" rpy="1.5708 0 0" />
+            <geometry>
+                <cylinder length="${forearm_length}" radius="0.02"/>
             </geometry>
         </collision>
     </link>
     <joint name="${prefix}jRightElbow_roty" type="revolute">
-        <origin xyz="0 -0.248 0" rpy="0 0 0"/>
+        <origin xyz="0 ${-float(forearm_length)} 0" rpy="0 0 0"/>
         <parent link="${prefix}RightForeArm"/>
         <child link="${prefix}RightForeArm_f1"/>
