Commit message: Refactor code structure for improved readability and maintainability

File: image_pose_tracking/config/right_arm_osim_shoulder.urdf.xacro (robot description, xacro)
@@ -1,4 +1,4 @@
 <?xml version="1.0"?>
-<robot xmlns:xacro="http://www.ros.org/wiki/xacro" name="upper_arm">
+<robot xmlns:xacro="http://www.ros.org/wiki/xacro" name="upper_arm_osim_shoulder">
     <xacro:arg name="robot_prefix" default=""/>
     <xacro:arg name="robot_color" default="blue"/>
@@ -11,4 +11,5 @@
     <xacro:property name="forearm_length" value="$(arg forearm_length)"/>
     <xacro:property name="forearm_com_y" value="${-float(forearm_length) / 2.0}"/>
+    <xacro:property name="mesh_dir" value="package://image_pose_tracking/meshes/human_subject_right_arm"/>
     <xacro:property name="color_code"  value="${
         '0.35 0.55 0.40 1' if color == 'green'
@@ -18,4 +19,7 @@
         <color rgba="${color_code}"/>
     </material>
+    <material name="torso_mesh_color">
+        <color rgba="0.76 0.66 0.58 1.0"/>
+    </material>
     <!-- <link name="camera_depth_optical_frame"/> -->
     <!-- <joint name="${prefix}world_to_shoulder" type="fixed">
@@ -24,40 +28,32 @@
         <origin xyz="-0.10466341 -0.122376    1.00400005" rpy="3.14 1.57 0"/>
     </joint> -->
-        <!-- === Trunk slab (torso) === -->
-    <link name="${prefix}Trunk">
-        <inertial>
-            <!-- Give it a small but nonzero mass to avoid NaNs -->
-            <mass value="5.0"/>
-            <origin xyz="0 0 0.20" rpy="0 0 0"/>
-            <!-- Rough, diagonal-dominant inertia for a 0.40 x 0.25 x 0.55 m box -->
-            <inertia ixx="0.5" iyy="0.8" izz="0.5" ixy="0" ixz="0" iyz="0"/>
-        </inertial>
-        <visual>
-            <origin xyz="0 0 0" rpy="0 0 0"/>
-            <!-- size = [width_x, depth_y, height_z] -->
-            <geometry>
-                <cylinder length="0.4" radius="0.02"/>
-            </geometry>
-            <material name="color">
-                <!-- subtle gray so the arm (green) stands out -->
-                <color rgba="0.6 0.6 0.6 1.0"/>
-            </material>
-        </visual>
-        <collision>
-            <origin xyz="0 0 0" rpy="0 0 0"/>
-            <geometry>
-                <cylinder length="0.4" radius="0.02"/>
-            </geometry>
-        </collision>
-    </link>
-    <joint name="${prefix}jShoulder_to_trunk" type="fixed">
-        <origin xyz="0 0 -0.20" rpy="0 0 0"/>
+    <!--
+        Static upper-torso visualization branch, matching the mesh xacro setup.
+        This fixed side branch is not inserted into the 7-DOF right-arm chain:
+        RightShoulder remains the root and the first commanded arm joint is
+        still jRightShoulder_elv_angle.
+    -->
+    <joint name="${prefix}jRightShoulder_to_UpperTorso" type="fixed">
+        <origin xyz="0 -0.073 -0.2" rpy="0 0 0"/>
         <parent link="${prefix}RightShoulder"/>
-        <child link="${prefix}Trunk"/>
-    </joint>
-    <!--  shoudler, 3DOF -->
+        <child link="${prefix}UpperTorso"/>
+    </joint>
+    <link name="${prefix}UpperTorso">
+        <visual>
+            <origin xyz="0 0 0" rpy="-1.5708 0 0"/>
+            <geometry>
+                <mesh filename="${mesh_dir}/UpperTrunk.stl" scale="0.58333333 1.03030303 1.03030303"/>
+            </geometry>
+            <material name="torso_mesh_color"/>
+        </visual>
+        <collision>
+            <origin xyz="0 0 0" rpy="-1.5708 0 0"/>
+            <geometry>
+                <box size="0.18 0.22 0.22"/>
+            </geometry>
+        </collision>
+    </link>
     <link name="${prefix}RightShoulder">
         <visual>
-			<!--box origin wrt jRightC7Shoulder. RPY rotated of pi/2.-->
             <origin xyz="0 0 0" rpy="0 0 0" />
             <geometry>
@@ -67,52 +63,70 @@
         </visual>
     </link>
-    <joint name="${prefix}jRightShoulder_rotx" type="revolute">
+    <!--
+        OSIM shoulder sequence from MOBL_ARMS_module5_scaleIK.osim:
+        shoulder0/elv_angle, shoulder1/shoulder_elv, shoulder1_r2=-elv_angle,
+        shoulder2/shoulder_rot. All joint origins remain at the shoulder center.
+    -->
+    <joint name="${prefix}jRightShoulder_elv_angle" type="revolute">
         <origin xyz="0 0 0" rpy="0 0 0"/>
         <parent link="${prefix}RightShoulder"/>
-        <child link="${prefix}RightUpperArm_f1"/>
-        <dynamics damping="0.1" friction="0.0"/>
-        <limit effort="30" velocity="1.0" lower="-2.35619" upper="1.5708" />
-        <axis xyz="1 0 0" />
-    </joint>
-    <link name="${prefix}RightUpperArm_f1">
-        <inertial>
-            <mass value="0"/>
-            <origin xyz="0 0 0" rpy="0 0 0" />
-            <inertia ixx="0" iyy="0" izz="0" ixy="0" ixz="0" iyz="0"/>
-        </inertial>
-    </link>
-    <joint name="${prefix}jRightShoulder_rotz" type="revolute">
-        <origin xyz="0 0 0" rpy="0 0 0"/>
-        <parent link="${prefix}RightUpperArm_f1"/>
-        <child link="${prefix}RightUpperArm_f2"/>
-        <dynamics damping="0.1" friction="0.0"/>
-        <limit effort="30" velocity="1.0" lower="-0.785398" upper="1.5708" />
-        <axis xyz="0 0 1" />
-    </joint>
-    <link name="${prefix}RightUpperArm_f2">
-        <inertial>
-            <mass value="0"/>
-            <origin xyz="0 0 0" rpy="0 0 0" />
-            <inertia ixx="0" iyy="0" izz="0" ixy="0" ixz="0" iyz="0"/>
-        </inertial>
-    </link>
-    <joint name="${prefix}jRightShoulder_roty" type="revolute">
-        <origin xyz="0 0 0" rpy="0 0 0"/>
-        <parent link="${prefix}RightUpperArm_f2"/>
+        <child link="${prefix}RightShoulder_elv_angle"/>
+        <dynamics damping="0.1" friction="0.0"/>
+        <limit effort="30" velocity="1.0" lower="-1.65806279" upper="2.26892803" />
+        <axis xyz="0.0048 0.99908918 0.04240001" />
+    </joint>
+    <link name="${prefix}RightShoulder_elv_angle">
+        <inertial>
+            <mass value="0"/>
+            <origin xyz="0 0 0" rpy="0 0 0" />
+            <inertia ixx="0" iyy="0" izz="0" ixy="0" ixz="0" iyz="0"/>
+        </inertial>
+    </link>
+    <joint name="${prefix}jRightShoulder_shoulder_elv" type="revolute">
+        <origin xyz="0 0 0" rpy="0 0 0"/>
+        <parent link="${prefix}RightShoulder_elv_angle"/>
+        <child link="${prefix}RightShoulder_shoulder_elv"/>
+        <dynamics damping="0.1" friction="0.0"/>
+        <limit effort="30" velocity="1.0" lower="0" upper="3.14159265" />
+        <axis xyz="-0.99826136 0.0023 0.05889802" />
+    </joint>
+    <link name="${prefix}RightShoulder_shoulder_elv">
+        <inertial>
+            <mass value="0"/>
+            <origin xyz="0 0 0" rpy="0 0 0" />
+            <inertia ixx="0" iyy="0" izz="0" ixy="0" ixz="0" iyz="0"/>
+        </inertial>
+    </link>
+    <joint name="${prefix}jRightShoulder_shoulder1_r2" type="revolute">
+        <origin xyz="0 0 0" rpy="0 0 0"/>
+        <parent link="${prefix}RightShoulder_shoulder_elv"/>
+        <child link="${prefix}RightShoulder_shoulder1_r2"/>
+        <dynamics damping="0.1" friction="0.0"/>
+        <limit effort="30" velocity="1.0" lower="-2.26892803" upper="1.65806279" />
+        <axis xyz="0.0048 0.99908918 0.04240001" />
+        <mimic joint="${prefix}jRightShoulder_elv_angle" multiplier="-1.0" offset="0.0"/>
+    </joint>
+    <link name="${prefix}RightShoulder_shoulder1_r2">
+        <inertial>
+            <mass value="0"/>
+            <origin xyz="0 0 0" rpy="0 0 0" />
+            <inertia ixx="0" iyy="0" izz="0" ixy="0" ixz="0" iyz="0"/>
+        </inertial>
+    </link>
+    <joint name="${prefix}jRightShoulder_shoulder_rot" type="revolute">
+        <origin xyz="0 0 0" rpy="0 0 0"/>
+        <parent link="${prefix}RightShoulder_shoulder1_r2"/>
         <child link="${prefix}RightUpperArm"/>
         <dynamics damping="0.1" friction="0.0"/>
-        <limit effort="30" velocity="1.0" lower="-1.5708" upper="1.5708" />
-        <axis xyz="0 1 0" />
-    </joint>
-    <!-- elbow, 3 dof -->
+        <limit effort="30" velocity="1.0" lower="-1.57079633" upper="2.09439510" />
+        <axis xyz="0.0048 0.99908918 0.04240001" />
+    </joint>
     <link name="${prefix}RightUpperArm">
         <inertial>
             <mass value="2.181"/>
-			<!--COM origin wrt jRightShoulder-->
             <origin xyz="0 ${upper_arm_com_y} 0" rpy="0 0 0" />
             <inertia ixx="0.020332" iyy="0.0013806" izz="0.020332" ixy="0" ixz="0" iyz="0"/>
         </inertial>
         <visual>
-			<!--box origin wrt jRightShoulder. RPY rotated of pi/2.-->
             <origin xyz="0 ${upper_arm_com_y} 0" rpy="1.5708 0 0" />
             <geometry>
@@ -122,5 +136,4 @@
         </visual>
         <collision>
-			<!--box origin wrt jRightShoulder. RPY rotated of pi/2.-->
             <origin xyz="0 ${upper_arm_com_y} 0" rpy="1.5708 0 0" />
             <geometry>
@@ -140,10 +153,8 @@
         <inertial>
             <mass value="1.454"/>
-			<!--COM origin wrt jRightElbow-->
             <origin xyz="0 ${forearm_com_y} 0" rpy="0 0 0" />
             <inertia ixx="0.008948" iyy="0.00040906" izz="0.008948" ixy="0" ixz="0" iyz="0"/>
         </inertial>
         <visual>
-			<!--box origin wrt jRightElbow. RPY rotated of pi/2.-->
             <origin xyz="0 ${forearm_com_y} 0" rpy="1.5708 0 0" />
             <geometry>
@@ -153,5 +164,4 @@
         </visual>
         <collision>
-			<!--box origin wrt jRightElbow. RPY rotated of pi/2.-->
             <origin xyz="0 ${forearm_com_y} 0" rpy="1.5708 0 0" />
             <geometry>
@@ -182,7 +192,6 @@
         </visual>
     </link>
-    <!-- wrist 2 dofs -->
     <joint name="${prefix}jRightWrist_rotx" type="revolute">
-        <origin xyz="0    0  0" rpy="0 0 0"/>
+        <origin xyz="0 0 0" rpy="0 0 0"/>
         <parent link="${prefix}RightForeArm_f1"/>
         <child link="${prefix}RightHand_f1"/>
@@ -209,21 +218,18 @@
         <inertial>
             <mass value="0.4362"/>
-			<!--COM origin wrt jRightWrist-->
-            <origin xyz="0    -0.05           0" rpy="0 0 0" />
+            <origin xyz="0 -0.05 0" rpy="0 0 0" />
             <inertia ixx="0.0015471" iyy="0.00073303" izz="0.0021165" ixy="0" ixz="0" iyz="0"/>
         </inertial>
         <visual>
-			<!--box origin wrt jRightWrist-->
-            <origin xyz="0    -0.05           0" rpy="0 0 0" />
-            <geometry>
-                <box size="0.06    0.085    0.03"/>
-            </geometry>
-            <material name="color"/>
-        </visual>
-        <collision>
-			<!--box origin wrt jRightWrist-->
-            <origin xyz="0    -0.05           0" rpy="0 0 0" />
-            <geometry>
-                <box size="0.04     0.133    0.133"/>
+            <origin xyz="0 -0.05 0" rpy="0 0 0" />
+            <geometry>
+                <box size="0.06 0.085 0.03"/>
+            </geometry>
+            <material name="color"/>
+        </visual>
+        <collision>
+            <origin xyz="0 -0.05 0" rpy="0 0 0" />
+            <geometry>
+                <box size="0.04 0.133 0.133"/>
             </geometry>
         </collision>
@@ -242,12 +248,10 @@
         </inertial>
         <visual>
-            <!--box origin wrt jRightWrist-->
-            <origin xyz="0   0           0" rpy="0 0 0" />
-            <geometry>
-                <box size="0     0    0"/>
-            </geometry>
-            <material name="color"/>
-        </visual>
-    </link>
-<!-- End of right arm configuration -->
+            <origin xyz="0 0 0" rpy="0 0 0" />
+            <geometry>
+                <box size="0 0 0"/>
+            </geometry>
+            <material name="color"/>
+        </visual>
+    </link>
 </robot>
