Commit message: Add per-subject arm geometry and grip calibration configuration
This commit introduces a new YAML configuration file that defines the arm lengths and grip offsets for multiple subjects. Each subject has specific parameters for upper arm length, forearm length, hand length, and grip offset, allowing for more accurate pose tracking and calibration in the image pose tracking system.

File: image_pose_tracking/config/right_arm_osim_shoulder_mesh.urdf.xacro (robot description, xacro)
@@ -79,5 +79,5 @@
                 <mesh filename="${mesh_dir}/RightShoulder.stl" scale="0.64444444 0.64444444 1.03030303"/>
             </geometry>
-            <material name="mesh_color"/>
+            <material name="color"/>
         </visual>
         <collision>
@@ -98,5 +98,5 @@
         <child link="${prefix}RightShoulder_elv_angle"/>
         <dynamics damping="0.1" friction="0.0"/>
-        <limit effort="30" velocity="1.0" lower="-1.65806279" upper="2.26892803"/>
+        <limit effort="30" velocity="1.0" lower="-1.04" upper="1.57"/>
         <axis xyz="0.0048 0.99908918 0.04240001"/>
     </joint>
@@ -113,5 +113,5 @@
         <child link="${prefix}RightShoulder_shoulder_elv"/>
         <dynamics damping="0.1" friction="0.0"/>
-        <limit effort="30" velocity="1.0" lower="0" upper="3.14159265"/>
+        <limit effort="30" velocity="1.0" lower="0" upper="2.094"/>
         <axis xyz="-0.99826136 0.0023 0.05889802"/>
     </joint>
@@ -128,5 +128,5 @@
         <child link="${prefix}RightShoulder_shoulder1_r2"/>
         <dynamics damping="0.1" friction="0.0"/>
-        <limit effort="30" velocity="1.0" lower="-2.26892803" upper="1.65806279"/>
+        <limit effort="30" velocity="1.0" lower="-1.04" upper="1.57"/>
         <axis xyz="0.0048 0.99908918 0.04240001"/>
         <mimic joint="${prefix}jRightShoulder_elv_angle" multiplier="-1.0" offset="0.0"/>
@@ -158,5 +158,5 @@
                 <mesh filename="${mesh_dir}/RightUpperArm.stl" scale="0.64444444 0.64444444 ${upper_arm_mesh_scale_z}"/>
             </geometry>
-            <material name="mesh_color"/>
+            <material name="color"/>
         </visual>
         <collision>
@@ -186,5 +186,5 @@
                 <mesh filename="${mesh_dir}/RightForeArm.stl" scale="0.61111111 0.61111111 ${forearm_mesh_scale_z}"/>
             </geometry>
-            <material name="mesh_color"/>
+            <material name="color"/>
         </visual>
         <collision>
@@ -215,5 +215,5 @@
         <child link="${prefix}RightHand_f1"/>
         <dynamics damping="0.1" friction="0.0"/>
-        <limit effort="30" velocity="1.0" lower="-1.5708" upper="1.5708"/>
+        <limit effort="30" velocity="1.0" lower="-1.047" upper="1.047"/>
         <axis xyz="1 0 0"/>
     </joint>
@@ -230,5 +230,5 @@
         <child link="${prefix}RightHand"/>
         <dynamics damping="0.1" friction="0.0"/>
-        <limit effort="30" velocity="1.0" lower="-0.723599" upper="0.549066"/>
+        <limit effort="30" velocity="1.0" lower="-0.52" upper="0.26"/>
         <axis xyz="0 0 1"/>
     </joint>
@@ -244,5 +244,5 @@
                 <mesh filename="${mesh_dir}/RightHand.stl" scale="0.9 ${hand_mesh_scale_y} 0.55555556"/>
             </geometry>
-            <material name="mesh_color"/>
+            <material name="color"/>
         </visual>
         <collision>
